File: coinPCB.sch (KiCad schematic (older format))
At the start: 12 parts, among them P1 CONN_01X08, P2 CONN_01X08, Q1 2N2222A, U1 TSOP38238, U2 DHT12

Commit message: added DHT12 symbol to project lib. Still uses DHT11 footprint
Parts:
- R1: symbol Device1:R -> Device:R
Changed lines of the file:
@@
 $EndComp
 $Comp
-L Device1:R R1
+L Device:R R1
 U 1 1 5CBCAB8A
 P 4650 3450

Commit message: updated symbols to new KiCad Library and digikey library
Parts:
- D1, D2, D3: symbol Device1:LED -> Device:LED
- R2, R3, R4: symbol Device1:R -> Device:R
- U2: symbol Sensor1:DHT11 -> DHT12:DHT12
Changed lines of the file:
@@
 P 3950 3000
 F 0 "U1" H 3855 3140 60  0000 L CNN
-F 1 "TSOP38238" H 4150 2600 60  0000 L CNN
+F 1 "TSOP38238" V 3750 2700 60  0000 L CNN
 F 2 "digikey-footprints:IR_Receiver_TSOP38238" H 4150 3200 60  0001 L CNN
 F 3 "http://www.vishay.com/docs/82491/tsop382.pdf" H 4150 3300 60  0001 L CNN
@@
 $EndComp
 $Comp
-L Device1:LED D1
+L Device:LED D1
 U 1 1 5CBCA17E
 P 5100 2850
@@
 $EndComp
 $Comp
-L Device1:R R2
+L Device:R R2
 U 1 1 5CBCAB0F
 P 5100 2050
@@
 +3.3V
 $Comp
-L Device1:R R3
+L Device:R R3
 U 1 1 5CBCDE03
 P 6000 2550
@@
 $EndComp
 $Comp
-L Device1:LED D2
+L Device:LED D2
 U 1 1 5CBCDE5F
 P 6000 3350
@@
 +3.3V
 $Comp
-L Device1:R R4
+L Device:R R4
 U 1 1 5CBCE8B3
 P 6600 2550
@@
 $EndComp
 $Comp
-L Device1:LED D3
+L Device:LED D3
 U 1 1 5CBCE91D
 P 6650 3300
@@
 	10400 950  10400 1050
 $Comp
-L Sensor1:DHT11 U2
+L DHT12:DHT12 U2
 U 1 1 5CBCDBB4
 P 7650 3100

Commit message: fixed all errors and should build correctly
Parts:
- R1, R2, R3, R4: footprint Resistor_THT:R_Axial_DIN0204_L3.6mm_D1.6mm_P1.90mm_Vertical -> Resistor_THT:R_Axial_DIN0204_L3.6mm_D1.6mm_P7.62mm_Horizontal
Connections:
- wire segments 44 -> 43
Changed lines of the file:
@@
-$EndComp
-$Comp
-L power:VCC #PWR02
-U 1 1 5CBCA4C7
-P 2550 2550
-F 0 "#PWR02" H 2550 2400 50  0001 C CNN
-F 1 "VCC" H 2550 2700 50  0000 C CNN
-F 2 "" H 2550 2550 50  0000 C CNN
-F 3 "" H 2550 2550 50  0000 C CNN
-	1    2550 2550
-	1    0    0    -1
 $EndComp
 $Comp
@@
 F 0 "R2" V 5180 2050 50  0000 C CNN
 F 1 "100" V 5100 2050 50  0000 C CNN
-F 2 "Resistor_THT:R_Axial_DIN0204_L3.6mm_D1.6mm_P1.90mm_Vertical" V 5030 2050 50  0001 C CNN
+F 2 "Resistor_THT:R_Axial_DIN0204_L3.6mm_D1.6mm_P7.62mm_Horizontal" V 5030 2050 50  0001 C CNN
 F 3 "" H 5100 2050 50  0000 C CNN
 	1    5100 2050
@@
 F 0 "R1" V 4730 3450 50  0000 C CNN
 F 1 "1K" V 4650 3450 50  0000 C CNN
-F 2 "Resistor_THT:R_Axial_DIN0204_L3.6mm_D1.6mm_P1.90mm_Vertical" V 4580 3450 50  0001 C CNN
+F 2 "Resistor_THT:R_Axial_DIN0204_L3.6mm_D1.6mm_P7.62mm_Horizontal" V 4580 3450 50  0001 C CNN
 F 3 "" H 4650 3450 50  0000 C CNN
 	1    4650 3450
@@
 	9350 1250 9450 1250
 Wire Wire Line
-	9350 1050 9450 1050
-Wire Wire Line
 	3100 3100 3650 3100
 Wire Wire Line
@@
 Wire Wire Line
 	10300 1750 10400 1750
-Text Label 2800 2550 0    60   ~ 0
-+3.3V
-Wire Wire Line
-	2550 2550 2800 2550
 Text Label 3100 3100 0    60   ~ 0
 D5
@@
 F 0 "R3" V 6080 2550 50  0000 C CNN
 F 1 "100" V 6000 2550 50  0000 C CNN
-F 2 "Resistor_THT:R_Axial_DIN0204_L3.6mm_D1.6mm_P1.90mm_Vertical" V 5930 2550 50  0001 C CNN
+F 2 "Resistor_THT:R_Axial_DIN0204_L3.6mm_D1.6mm_P7.62mm_Horizontal" V 5930 2550 50  0001 C CNN
 F 3 "" H 6000 2550 50  0000 C CNN
 	1    6000 2550
@@
 F 0 "R4" V 6680 2550 50  0000 C CNN
 F 1 "100" V 6600 2550 50  0000 C CNN
-F 2 "Resistor_THT:R_Axial_DIN0204_L3.6mm_D1.6mm_P1.90mm_Vertical" V 6530 2550 50  0001 C CNN
+F 2 "Resistor_THT:R_Axial_DIN0204_L3.6mm_D1.6mm_P7.62mm_Horizontal" V 6530 2550 50  0001 C CNN
 F 3 "" H 6600 2550 50  0000 C CNN
 	1    6600 2550
@@
 $EndComp
 Wire Wire Line
-	7150 3100 7450 3100
+	7150 3100 7350 3100
+Wire Wire Line
+	9350 1050 9450 1050
 $EndSCHEMATC

Commit message: fixed schematic errors, including taking out 1k resitor from D3 because that pin as pull-up resistor arleady, and running D4 and D8 to ground
Parts:
- removed R1: 1K, Resistor_THT:R_Axial_DIN0204_L3.6mm_D1.6mm_P7.62mm_Horizontal, symbol Device:R
Connections:
- wire segments 43 -> 41
Changed lines of the file:
@@
 	-1   0    0    -1
 $EndComp
-Text Label 9350 1050 2    60   ~ 0
-+5V
 Text Label 9350 1150 2    60   ~ 0
 GND
@@
 Text Label 9350 1750 2    60   ~ 0
 TX
-Text Label 10400 1050 0    60   ~ 0
-+3.3V
 Text Label 10400 1150 0    60   ~ 0
 D8
@@
 $EndComp
 $Comp
-L power:GND #PWR03
-U 1 1 5CBCA4E1
-P 9200 1850
-F 0 "#PWR03" H 9200 1600 50  0001 C CNN
-F 1 "GND" H 9200 1700 50  0000 C CNN
-F 2 "" H 9200 1850 50  0000 C CNN
-F 3 "" H 9200 1850 50  0000 C CNN
-	1    9200 1850
-	1    0    0    -1
-$EndComp
-$Comp
 L Device:R R2
 U 1 1 5CBCAB0F
@@
 $EndComp
 $Comp
-L Device:R R1
-U 1 1 5CBCAB8A
-P 4650 3450
-F 0 "R1" V 4730 3450 50  0000 C CNN
-F 1 "1K" V 4650 3450 50  0000 C CNN
-F 2 "Resistor_THT:R_Axial_DIN0204_L3.6mm_D1.6mm_P7.62mm_Horizontal" V 4580 3450 50  0001 C CNN
-F 3 "" H 4650 3450 50  0000 C CNN
-	1    4650 3450
-	0    1    1    0
-$EndComp
-Text Label 5200 1650 2    60   ~ 0
-+5V
-$Comp
 L power:GND #PWR04
 U 1 1 5CBCAE77
@@
 	1    0    0    -1
 $EndComp
-Text Label 4300 3450 2    60   ~ 0
+Text Label 4700 3450 2    60   ~ 0
 D3
 Wire Notes Line
@@
 	8500 2100 11200 2100
 Wire Wire Line
-	5200 1650 5100 1650
-Wire Wire Line
 	5100 1650 5100 1900
 Wire Wire Line
@@
 	3100 3100 3650 3100
 Wire Wire Line
-	4300 3450 4500 3450
-Wire Wire Line
-	4800 3450 4850 3450
+	4700 3450 4850 3450
 Wire Wire Line
 	9450 1650 9350 1650
 Wire Wire Line
 	9450 1750 9350 1750
-Wire Wire Line
-	10300 1050 10400 1050
 Wire Wire Line
 	10300 1150 10400 1150
@@
 Text Label 3100 3100 0    60   ~ 0
 D5
-Text Label 3950 2200 0    60   ~ 0
-+3.3V
-Text Label 5900 1900 0    60   ~ 0
-+3.3V
 $Comp
 L Device:R R3
 U 1 1 5CBCDE03
+P 6000 3350
+F 0 "R3" V 6080 3350 50  0000 C CNN
+F 1 "100" V 6000 3350 50  0000 C CNN
+F 2 "Resistor_THT:R_Axial_DIN0204_L3.6mm_D1.6mm_P7.62mm_Horizontal" V 5930 3350 50  0001 C CNN
+F 3 "" H 6000 3350 50  0000 C CNN
+	1    6000 3350
+	1    0    0    -1
+$EndComp
+$Comp
+L Device:LED D2
+U 1 1 5CBCDE5F
 P 6000 2550
-F 0 "R3" V 6080 2550 50  0000 C CNN
-F 1 "100" V 6000 2550 50  0000 C CNN
-F 2 "Resistor_THT:R_Axial_DIN0204_L3.6mm_D1.6mm_P7.62mm_Horizontal" V 5930 2550 50  0001 C CNN
+F 0 "D2" H 6000 2650 50  0000 C CNN
+F 1 "LED" H 6000 2450 50  0000 C CNN
+F 2 "digikey-footprints:LED_3mm_Radial" H 6000 2550 50  0001 C CNN
 F 3 "" H 6000 2550 50  0000 C CNN
 	1    6000 2550
-	1    0    0    -1
-$EndComp
-$Comp
-L Device:LED D2
-U 1 1 5CBCDE5F
-P 6000 3350
-F 0 "D2" H 6000 3450 50  0000 C CNN
-F 1 "LED" H 6000 3250 50  0000 C CNN
-F 2 "digikey-footprints:LED_3mm_Radial" H 6000 3350 50  0001 C CNN
-F 3 "" H 6000 3350 50  0000 C CNN
-	1    6000 3350
 	0    -1   -1   0
 $EndComp
-Text Label 6000 4000 0    60   ~ 0
+Text Label 5900 1900 0    60   ~ 0
 D8
-Text Label 6550 1900 0    60   ~ 0
-+3.3V
 $Comp
 L Device:R R4
 U 1 1 5CBCE8B3
+P 6650 3300
+F 0 "R4" V 6730 3300 50  0000 C CNN
+F 1 "100" V 6650 3300 50  0000 C CNN
+F 2 "Resistor_THT:R_Axial_DIN0204_L3.6mm_D1.6mm_P7.62mm_Horizontal" V 6580 3300 50  0001 C CNN
+F 3 "" H 6650 3300 50  0000 C CNN
+	1    6650 3300
+	1    0    0    -1
+$EndComp
+$Comp
+L Device:LED D3
+U 1 1 5CBCE91D
 P 6600 2550
-F 0 "R4" V 6680 2550 50  0000 C CNN
-F 1 "100" V 6600 2550 50  0000 C CNN
-F 2 "Resistor_THT:R_Axial_DIN0204_L3.6mm_D1.6mm_P7.62mm_Horizontal" V 6530 2550 50  0001 C CNN
+F 0 "D3" H 6600 2650 50  0000 C CNN
+F 1 "LED" H 6600 2450 50  0000 C CNN
+F 2 "digikey-footprints:LED_3mm_Radial" H 6600 2550 50  0001 C CNN
 F 3 "" H 6600 2550 50  0000 C CNN
 	1    6600 2550
-	1    0    0    -1
-$EndComp
-$Comp
-L Device:LED D3
-U 1 1 5CBCE91D
-P 6650 3300
-F 0 "D3" H 6650 3400 50  0000 C CNN
-F 1 "LED" H 6650 3200 50  0000 C CNN
-F 2 "digikey-footprints:LED_3mm_Radial" H 6650 3300 50  0001 C CNN
-F 3 "" H 6650 3300 50  0000 C CNN
-	1    6650 3300
 	0    -1   -1   0
 $EndComp
-Text Label 6650 3900 2    60   ~ 0
+Text Label 6550 1900 2    60   ~ 0
 D4
 Wire Wire Line
@@
 	6600 3150 6650 3150
 Wire Wire Line
-	6000 3500 6000 4000
-Wire Wire Line
 	6650 3450 6650 3900
-Text Label 7650 2000 0    60   ~ 0
-+3.3V
 $Comp
 L power:GND #PWR05
@@
 	7950 3100 8350 3100
 Wire Wire Line
-	7650 2000 7650 2800
-Wire Wire Line
 	3950 2200 3950 2800
-Wire Wire Line
-	3950 3400 3950 4300
-Wire Wire Line
-	7150 3100 7150 4100
-Wire Wire Line
-	9200 1150 9200 1850
-Wire Wire Line
-	9200 1150 9450 1150
-Wire Wire Line
-	5150 4300 5150 3650
-$Comp
-L power:VCC #PWR0101
-U 1 1 5CBFEED3
-P 10400 950
-F 0 "#PWR0101" H 10400 800 50  0001 C CNN
-F 1 "VCC" H 10417 1123 50  0000 C CNN
-F 2 "" H 10400 950 50  0001 C CNN
-F 3 "" H 10400 950 50  0001 C CNN
-	1    10400 950
-	1    0    0    -1
-$EndComp
-Wire Wire Line
-	10400 950  10400 1050
 $Comp
 L DHT12:DHT12 U2
@@
 Wire Wire Line
 	7150 3100 7350 3100
+$Comp
+L power:GND #PWR0102
+U 1 1 5CCBD639
+P 6650 3900
+F 0 "#PWR0102" H 6650 3650 50  0001 C CNN
+F 1 "GND" H 6650 3750 50  0000 C CNN
+F 2 "" H 6650 3900 50  0000 C CNN
+F 3 "" H 6650 3900 50  0000 C CNN
+	1    6650 3900
+	1    0    0    -1
+$EndComp
+$Comp
+L power:GND #PWR0103
+U 1 1 5CCBD65C
+P 6000 4000
+F 0 "#PWR0103" H 6000 3750 50  0001 C CNN
+F 1 "GND" H 6000 3850 50  0000 C CNN
+F 2 "" H 6000 4000 50  0000 C CNN
+F 3 "" H 6000 4000 50  0000 C CNN
+	1    6000 4000
+	1    0    0    -1
+$EndComp
 Wire Wire Line
 	9350 1050 9450 1050
+Wire Wire Line
+	9350 1150 9450 1150
+$Comp
+L power:+5V #PWR0101
+U 1 1 5CCC81C0
+P 5100 1650
+F 0 "#PWR0101" H 5100 1500 50  0001 C CNN
+F 1 "+5V" H 5115 1823 50  0000 C CNN
+F 2 "" H 5100 1650 50  0001 C CNN
+F 3 "" H 5100 1650 50  0001 C CNN
+	1    5100 1650
+	1    0    0    -1
+$EndComp
+$Comp
+L power:+3.3V #PWR0104
+U 1 1 5CCC8281
+P 3950 2200
+F 0 "#PWR0104" H 3950 2050 50  0001 C CNN
+F 1 "+3.3V" H 3965 2373 50  0000 C CNN
+F 2 "" H 3950 2200 50  0001 C CNN
+F 3 "" H 3950 2200 50  0001 C CNN
+	1    3950 2200
+	1    0    0    -1
+$EndComp
+$Comp
+L power:+3.3V #PWR0105
+U 1 1 5CCC8FF6
+P 7650 2000
+F 0 "#PWR0105" H 7650 1850 50  0001 C CNN
+F 1 "+3.3V" H 7665 2173 50  0000 C CNN
+F 2 "" H 7650 2000 50  0001 C CNN
+F 3 "" H 7650 2000 50  0001 C CNN
+	1    7650 2000
+	1    0    0    -1
+$EndComp
+Wire Wire Line
+	7150 3100 7150 4100
+Wire Wire Line
+	7650 2000 7650 2800
+Wire Wire Line
+	10300 1050 10400 1050
+Text Label 10400 1050 0    60   ~ 0
++3.3V
+Text Label 9350 1050 2    60   ~ 0
++5V
+$Comp
+L power:+5V #PWR0106
+U 1 1 5CCD434C
+P 9450 900
+F 0 "#PWR0106" H 9450 750 50  0001 C CNN
+F 1 "+5V" H 9465 1073 50  0000 C CNN
+F 2 "" H 9450 900 50  0001 C CNN
+F 3 "" H 9450 900 50  0001 C CNN
+	1    9450 900
+	1    0    0    -1
+$EndComp
+$Comp
+L power:VCC #PWR0107
+U 1 1 5CCD4A83
+P 10300 850
+F 0 "#PWR0107" H 10300 700 50  0001 C CNN
+F 1 "VCC" H 10317 1023 50  0000 C CNN
+F 2 "" H 10300 850 50  0001 C CNN
+F 3 "" H 10300 850 50  0001 C CNN
+	1    10300 850
+	1    0    0    -1
+$EndComp
+Wire Wire Line
+	10300 850  10300 1050
+Connection ~ 10300 1050
+Wire Wire Line
+	9450 900  9450 1050
+Connection ~ 9450 1050
+Wire Wire Line
+	3950 4300 3950 3400
+Wire Wire Line
+	6000 4000 6000 3500
+Wire Wire Line
+	5150 4300 5150 3650
 $EndSCHEMATC

Commit message: began laying out v0.2 with digikeyfootprins
Parts:
- renumbered D2 to D10, D3 to D11, D1 to D9, R2 to R1, R3 to R2, R4 to R3
Changed lines of the file:
@@
 $EndComp
 $Comp
-L Device:LED D1
+L Device:LED D9
 U 1 1 5CBCA17E
 P 5100 2850
-F 0 "D1" H 5100 2950 50  0000 C CNN
+F 0 "D9" H 5100 2950 50  0000 C CNN
 F 1 "LED" H 5100 2750 50  0000 C CNN
 F 2 "digikey-footprints:LED_3mm_Radial" H 5100 2850 50  0001 C CNN
@@
 $EndComp
 $Comp
-L power:GND #PWR01
+L power:GND #PWR02
 U 1 1 5CBCA465
 P 3950 4300
-F 0 "#PWR01" H 3950 4050 50  0001 C CNN
+F 0 "#PWR02" H 3950 4050 50  0001 C CNN
 F 1 "GND" H 3950 4150 50  0000 C CNN
 F 2 "" H 3950 4300 50  0000 C CNN
@@
 $EndComp
 $Comp
-L Device:R R2
+L Device:R R1
 U 1 1 5CBCAB0F
 P 5100 2050
-F 0 "R2" V 5180 2050 50  0000 C CNN
+F 0 "R1" V 5180 2050 50  0000 C CNN
 F 1 "100" V 5100 2050 50  0000 C CNN
 F 2 "Resistor_THT:R_Axial_DIN0204_L3.6mm_D1.6mm_P7.62mm_Horizontal" V 5030 2050 50  0001 C CNN
@@
 D5
 $Comp
-L Device:R R3
+L Device:R R2
 U 1 1 5CBCDE03
 P 6000 3350
-F 0 "R3" V 6080 3350 50  0000 C CNN
+F 0 "R2" V 6080 3350 50  0000 C CNN
 F 1 "100" V 6000 3350 50  0000 C CNN
 F 2 "Resistor_THT:R_Axial_DIN0204_L3.6mm_D1.6mm_P7.62mm_Horizontal" V 5930 3350 50  0001 C CNN
@@
 $EndComp
 $Comp
-L Device:LED D2
+L Device:LED D10
 U 1 1 5CBCDE5F
 P 6000 2550
-F 0 "D2" H 6000 2650 50  0000 C CNN
+F 0 "D10" H 6000 2650 50  0000 C CNN
 F 1 "LED" H 6000 2450 50  0000 C CNN
 F 2 "digikey-footprints:LED_3mm_Radial" H 6000 2550 50  0001 C CNN
@@
 D8
 $Comp
-L Device:R R4
+L Device:R R3
 U 1 1 5CBCE8B3
 P 6650 3300
-F 0 "R4" V 6730 3300 50  0000 C CNN
+F 0 "R3" V 6730 3300 50  0000 C CNN
 F 1 "100" V 6650 3300 50  0000 C CNN
 F 2 "Resistor_THT:R_Axial_DIN0204_L3.6mm_D1.6mm_P7.62mm_Horizontal" V 6580 3300 50  0001 C CNN
@@
 $EndComp
 $Comp
-L Device:LED D3
+L Device:LED D11
 U 1 1 5CBCE91D
 P 6600 2550
-F 0 "D3" H 6600 2650 50  0000 C CNN
+F 0 "D11" H 6600 2650 50  0000 C CNN
 F 1 "LED" H 6600 2450 50  0000 C CNN
 F 2 "digikey-footprints:LED_3mm_Radial" H 6600 2550 50  0001 C CNN
@@
 	6650 3450 6650 3900
 $Comp
-L power:GND #PWR05
+L power:GND #PWR07
 U 1 1 5CBCE031
 P 7150 4100
-F 0 "#PWR05" H 7150 3850 50  0001 C CNN
+F 0 "#PWR07" H 7150 3850 50  0001 C CNN
 F 1 "GND" H 7150 3950 50  0000 C CNN
 F 2 "" H 7150 4100 50  0000 C CNN
@@
 	7150 3100 7350 3100
 $Comp
-L power:GND #PWR0102
+L power:GND #PWR06
 U 1 1 5CCBD639
 P 6650 3900
-F 0 "#PWR0102" H 6650 3650 50  0001 C CNN
+F 0 "#PWR06" H 6650 3650 50  0001 C CNN
 F 1 "GND" H 6650 3750 50  0000 C CNN
 F 2 "" H 6650 3900 50  0000 C CNN
@@
 $EndComp
 $Comp
-L power:GND #PWR0103
+L power:GND #PWR05
 U 1 1 5CCBD65C
 P 6000 4000
-F 0 "#PWR0103" H 6000 3750 50  0001 C CNN
+F 0 "#PWR05" H 6000 3750 50  0001 C CNN
 F 1 "GND" H 6000 3850 50  0000 C CNN
 F 2 "" H 6000 4000 50  0000 C CNN
@@
 	9350 1150 9450 1150
 $Comp
-L power:+5V #PWR0101
+L power:+5V #PWR03
 U 1 1 5CCC81C0
 P 5100 1650
-F 0 "#PWR0101" H 5100 1500 50  0001 C CNN
+F 0 "#PWR03" H 5100 1500 50  0001 C CNN
 F 1 "+5V" H 5115 1823 50  0000 C CNN
 F 2 "" H 5100 1650 50  0001 C CNN
@@
 $EndComp
 $Comp
-L power:+3.3V #PWR0104
+L power:+3.3V #PWR01
 U 1 1 5CCC8281
 P 3950 2200
-F 0 "#PWR0104" H 3950 2050 50  0001 C CNN
+F 0 "#PWR01" H 3950 2050 50  0001 C CNN
 F 1 "+3.3V" H 3965 2373 50  0000 C CNN
 F 2 "" H 3950 2200 50  0001 C CNN
@@
 $EndComp
 $Comp
-L power:+3.3V #PWR0105
+L power:+3.3V #PWR08
 U 1 1 5CCC8FF6
 P 7650 2000
-F 0 "#PWR0105" H 7650 1850 50  0001 C CNN
+F 0 "#PWR08" H 7650 1850 50  0001 C CNN
 F 1 "+3.3V" H 7665 2173 50  0000 C CNN
 F 2 "" H 7650 2000 50  0001 C CNN
@@
 +5V
 $Comp
-L power:+5V #PWR0106
+L power:+5V #PWR09
 U 1 1 5CCD434C
 P 9450 900
-F 0 "#PWR0106" H 9450 750 50  0001 C CNN
+F 0 "#PWR09" H 9450 750 50  0001 C CNN
 F 1 "+5V" H 9465 1073 50  0000 C CNN
 F 2 "" H 9450 900 50  0001 C CNN
@@
 $EndComp
 $Comp
-L power:VCC #PWR0107
+L power:VCC #PWR010
 U 1 1 5CCD4A83
 P 10300 850
-F 0 "#PWR0107" H 10300 700 50  0001 C CNN
+F 0 "#PWR010" H 10300 700 50  0001 C CNN
 F 1 "VCC" H 10317 1023 50  0000 C CNN
 F 2 "" H 10300 850 50  0001 C CNN

Commit message: finished initial PCB trace layout and added the copper backplane as well as fixed the digi-key model of the IR_LED_TSAL_6100 to have the Cathode be the square pad.
Parts:
- D9: footprint digikey-footprints:LED_3mm_Radial -> digikey-footprints:LED_IR_TSAL6100; symbol Device:LED -> dk_Infrared-UV-Visible-Emitters:TSAL6100
Connections:
- net labels removed: VCC
Changed lines of the file:
@@
 $EndComp
 $Comp
-L Device:LED D9
+L dk_Infrared-UV-Visible-Emitters:TSAL6100 D9
 U 1 1 5CBCA17E
-P 5100 2850
-F 0 "D9" H 5100 2950 50  0000 C CNN
-F 1 "LED" H 5100 2750 50  0000 C CNN
-F 2 "digikey-footprints:LED_3mm_Radial" H 5100 2850 50  0001 C CNN
-F 3 "" H 5100 2850 50  0000 C CNN
-	1    5100 2850
-	0    -1   -1   0
+P 5100 2800
+F 0 "D9" H 5100 2900 50  0000 C CNN
+F 1 "LED" H 5100 2700 50  0000 C CNN
+F 2 "digikey-footprints:LED_IR_TSAL6100" H 5100 2800 50  0001 C CNN
+F 3 "" H 5100 2800 50  0000 C CNN
+	1    5100 2800
+	0    1    1    0
 $EndComp
 $Comp
@@
 	5100 1650 5100 1900
 Wire Wire Line
-	5100 2200 5100 2700
-Wire Wire Line
-	5100 3000 5100 3250
-Wire Wire Line
 	5100 3250 5150 3250
 Wire Wire Line
@@
 	1    0    0    -1
 $EndComp
-$Comp
-L power:VCC #PWR010
-U 1 1 5CCD4A83
+Wire Wire Line
+	10300 850  10300 1050
+Connection ~ 10300 1050
+Wire Wire Line
+	9450 900  9450 1050
+Connection ~ 9450 1050
+Wire Wire Line
+	3950 4300 3950 3400
+Wire Wire Line
+	6000 4000 6000 3500
+Wire Wire Line
+	5150 4300 5150 3650
+$Comp
+L power:+3.3V #PWR0101
+U 1 1 5CCBFCD6
 P 10300 850
-F 0 "#PWR010" H 10300 700 50  0001 C CNN
-F 1 "VCC" H 10317 1023 50  0000 C CNN
+F 0 "#PWR0101" H 10300 700 50  0001 C CNN
+F 1 "+3.3V" H 10315 1023 50  0000 C CNN
 F 2 "" H 10300 850 50  0001 C CNN
 F 3 "" H 10300 850 50  0001 C CNN
@@
 $EndComp
 Wire Wire Line
-	10300 850  10300 1050
-Connection ~ 10300 1050
-Wire Wire Line
-	9450 900  9450 1050
-Connection ~ 9450 1050
-Wire Wire Line
-	3950 4300 3950 3400
-Wire Wire Line
-	6000 4000 6000 3500
-Wire Wire Line
-	5150 4300 5150 3650
+	5100 3250 5100 3000
+Wire Wire Line
+	5100 2700 5100 2200
 $EndSCHEMATC

Commit message: added final resitor values to 5v line
Parts:
- R1: value 100 -> 35
Changed lines of the file:
@@
 P 5100 2050
 F 0 "R1" V 5180 2050 50  0000 C CNN
-F 1 "100" V 5100 2050 50  0000 C CNN
+F 1 "35" V 5100 2050 50  0000 C CNN
 F 2 "Resistor_THT:R_Axial_DIN0204_L3.6mm_D1.6mm_P7.62mm_Horizontal" V 5030 2050 50  0001 C CNN
 F 3 "" H 5100 2050 50  0000 C CNN
