File: coinPCB.sch (KiCad schematic (older format))
At the start: 11 parts, among them P1 CONN_01X08, P2 CONN_01X08, Q1 2N2222A, U1 TSOP38238, U2 DHT12

Commit message: finalized moving footprint and symbol libraries to shared place to work with the KiCAD Dockerfile.
Parts:
- P1, P2: symbol coinPCB-rescue:CONN_01X08-cointest-rescue-coinPCB-rescue -> D1_mini:CONN_01X08
Changed lines of the file:
@@
 EESchema Schematic File Version 4
-LIBS:coinPCB-cache
-EELAYER 26 0
+EELAYER 29 0
 EELAYER END
 $Descr A4 11693 8268
@@
 $EndDescr
 $Comp
-L coinPCB-rescue:CONN_01X08-cointest-rescue-coinPCB-rescue P1
+L D1_mini:CONN_01X08 P1
 U 1 1 5763EB78
 P 9650 1400
@@
 $EndComp
 $Comp
-L coinPCB-rescue:CONN_01X08-cointest-rescue-coinPCB-rescue P2
+L D1_mini:CONN_01X08 P2
 U 1 1 5763EBF2
 P 10100 1400
@@
 Wire Wire Line
 	10300 850  10300 1050
-Connection ~ 10300 1050
 Wire Wire Line
 	9450 900  9450 1050
-Connection ~ 9450 1050
 Wire Wire Line
 	3950 4300 3950 3400
