File: coinPCB.kicad_pcb (KiCad board)
At the start: 2 copper layers, 50.8 x 50.8 mm, 11 parts, among them P1 CONN_01X08, P2 CONN_01X08, Q1 2N2222A, U1 TSOP38238, U2 DHT12

Commit message: Moved over IR TX pin to D0 because of issues with D3 Pull-up at boot time.
Parts:
- R1: value 100 -> 35
- moved Q1 2.78 mm to (123.1, 93.7), turned to 0 degrees
Connections:
- P1 pad 4: /D3 -> (no net)
- P1 pad 7: /RX -> (no net)
- P1 pad 8: /TX -> (no net)
- P2 pad 3: /D7 -> (no net)
- P2 pad 4: /D6 -> (no net)
- P2 pad 7: /A0 -> (no net)
- P2 pad 8: /RST -> (no net)
- Q1 pad 2: /D3 -> /D0
Routing:
- net /D0: track 0.00 -> 32.9 mm
- net /D3: track 9.27 -> 0.00 mm
- net Net-(D9-Pad2): track 7.68 -> 10.4 mm
- net (no net): track 0.00 -> 0.55 mm
Other:
- board text added: "v0.3"
- board text removed: "v0.2"

Commit message: v0.3 update with gbr files
Connections:
- P1 pad 4: (no net) -> /D3
- P1 pad 7: (no net) -> /RX
- P1 pad 8: (no net) -> /TX
- P2 pad 3: (no net) -> /D7
- P2 pad 4: (no net) -> /D6
- P2 pad 7: (no net) -> /A0
- P2 pad 8: (no net) -> /RST
Routing:
- net /D3: track 0.00 -> 0.55 mm
- net (no net): track 0.55 -> 0.00 mm
